Commit message: Add only model branch

File: dobot_cr16.urdf.xacro (robot description, xacro)
@@ -25,5 +25,5 @@
       <geometry>
         <mesh
-          filename="package://dobot_description/meshes/cr16/base_link.STL"  />
+          filename="./meshes/base_link.STL"  />
       </geometry>
       <material
@@ -39,5 +39,5 @@
       <geometry>
         <mesh
-          filename="package://dobot_description/meshes/cr16/base_link.STL"/>
+          filename="./meshes/base_link.STL"/>
           <box size="1.1 1.8 0.3"/>
       </geometry>
@@ -66,19 +66,19 @@
       <geometry>
         <mesh
-          filename="package://dobot_description/meshes/cr16/Link1.STL" />
-      </geometry>
-      <material
-        name="">
-        <color
-          rgba="1 1 1 1" />
-      </material>
-    </visual>
-    <collision>
-      <origin
-        xyz="0 0 0"
-        rpy="0 0 0" />
-      <geometry>
-        <mesh
-          filename="package://dobot_description/meshes/cr16/Link1.STL" />
+          filename="./meshes/Link1.STL" />
+      </geometry>
+      <material
+        name="">
+        <color
+          rgba="1 1 1 1" />
+      </material>
+    </visual>
+    <collision>
+      <origin
+        xyz="0 0 0"
+        rpy="0 0 0" />
+      <geometry>
+        <mesh
+          filename="./meshes/Link1.STL" />
       </geometry>
     </collision>
@@ -124,19 +124,19 @@
       <geometry>
         <mesh
-          filename="package://dobot_description/meshes/cr16/Link2.STL"  />
-      </geometry>
-      <material
-        name="">
-        <color
-          rgba="1 1 1 1" />
-      </material>
-    </visual>
-    <collision>
-      <origin
-        xyz="0 0 0"
-        rpy="0 0 0" />
-      <geometry>
-        <mesh
-          filename="package://dobot_description/meshes/cr16/Link2.STL" />
+          filename="./meshes/Link2.STL"  />
+      </geometry>
+      <material
+        name="">
+        <color
+          rgba="1 1 1 1" />
+      </material>
+    </visual>
+    <collision>
+      <origin
+        xyz="0 0 0"
+        rpy="0 0 0" />
+      <geometry>
+        <mesh
+          filename="./meshes/Link2.STL" />
       </geometry>
     </collision>
@@ -182,19 +182,19 @@
       <geometry>
         <mesh
-          filename="package://dobot_description/meshes/cr16/Link3.STL" />
-      </geometry>
-      <material
-        name="">
-        <color
-          rgba="1 1 1 1" />
-      </material>
-    </visual>
-    <collision>
-      <origin
-        xyz="0 0 0"
-        rpy="0 0 0" />
-      <geometry>
-        <mesh
-          filename="package://dobot_description/meshes/cr16/Link3.STL" />
+          filename="./meshes/Link3.STL" />
+      </geometry>
+      <material
+        name="">
+        <color
+          rgba="1 1 1 1" />
+      </material>
+    </visual>
+    <collision>
+      <origin
+        xyz="0 0 0"
+        rpy="0 0 0" />
+      <geometry>
+        <mesh
+          filename="./meshes/Link3.STL" />
       </geometry>
     </collision>
@@ -240,19 +240,19 @@
       <geometry>
         <mesh
-          filename="package://dobot_description/meshes/cr16/Link4.STL" />
-      </geometry>
-      <material
-        name="">
-        <color
-          rgba="1 1 1 1" />
-      </material>
-    </visual>
-    <collision>
-      <origin
-        xyz="0 0 0"
-        rpy="0 0 0" />
-      <geometry>
-        <mesh
-          filename="package://dobot_description/meshes/cr16/Link4.STL" />
+          filename="./meshes/Link4.STL" />
+      </geometry>
+      <material
+        name="">
+        <color
+          rgba="1 1 1 1" />
+      </material>
+    </visual>
+    <collision>
+      <origin
+        xyz="0 0 0"
+        rpy="0 0 0" />
+      <geometry>
+        <mesh
+          filename="./meshes/Link4.STL" />
       </geometry>
     </collision>
@@ -298,19 +298,19 @@
       <geometry>
         <mesh
-          filename="package://dobot_description/meshes/cr16/Link5.STL" />
-      </geometry>
-      <material
-        name="">
-        <color
-          rgba="1 1 1 1" />
-      </material>
-    </visual>
-    <collision>
-      <origin
-        xyz="0 0 0"
-        rpy="0 0 0" />
-      <geometry>
-        <mesh
-          filename="package://dobot_description/meshes/cr16/Link5.STL" />
+          filename="./meshes/Link5.STL" />
+      </geometry>
+      <material
+        name="">
+        <color
+          rgba="1 1 1 1" />
+      </material>
+    </visual>
+    <collision>
+      <origin
+        xyz="0 0 0"
+        rpy="0 0 0" />
+      <geometry>
+        <mesh
+          filename="./meshes/Link5.STL" />
       </geometry>
     </collision>
@@ -356,19 +356,19 @@
       <geometry>
         <mesh
-          filename="package://dobot_description/meshes/cr16/Link6.STL"/>
-      </geometry>
-      <material
-        name="">
-        <color
-          rgba="1 1 1 1" />
-      </material>
-    </visual>
-    <collision>
-      <origin
-        xyz="0 0 0"
-        rpy="0 0 0" />
-      <geometry>
-        <mesh
-          filename="package://dobot_description/meshes/cr16/Link6.STL" />
+          filename="./meshes/Link6.STL"/>
+      </geometry>
+      <material
+        name="">
+        <color
+          rgba="1 1 1 1" />
+      </material>
+    </visual>
+    <collision>
+      <origin
+        xyz="0 0 0"
+        rpy="0 0 0" />
+      <geometry>
+        <mesh
+          filename="./meshes/Link6.STL" />
       </geometry>
     </collision>
